Commit message: Bringing up to date with what's on the robot

File: config/udv.urdf (robot description, URDF)
Before this commit: robot udv, 4 links, 3 joints
Links:
- added link camera_link; visual cylinder length=0.05 radius=0.05
Joints:
- added joint base_to_camera_link: type fixed, parent base_link, child camera_link, origin xyz=0.149225 0 0.3 rpy=0 0 3.14159265359
